File: KiCAD/sandbox_enlik/sandbox_enlik.kicad_pcb (KiCad board)
At the start: 2 copper layers, 0 parts

Commit message: added new reference
Parts:
- added REF**: KSA_Tactile_SPST, Button_Switch_THT:KSA_Tactile_SPST, F.Cu at (168.0, 69.2)
- added REF**: BatteryHolder_Keystone_107_1x23mm, Battery:BatteryHolder_Keystone_107_1x23mm, F.Cu at (183.4, 82.5)
- added REF**: BatteryHolder_Keystone_107_1x23mm, Battery:BatteryHolder_Keystone_107_1x23mm, F.Cu at (196.9, 110.0)
